Commit message: Added crazyflie.urdf from gym-pybullet-drones to position_box.py

File: Crazyflie_Simulation/solid/assets/box.urdf (robot description, URDF)
Before this commit: robot box, 1 links, 0 joints
Links:
- link baseLink: geometry collision box size=0.07 0.07 0.07; visual mesh filename=./cf2.dae scale=1 1 1
